File: keeb.kicad_sch (KiCad schematic)
At the start: 321 parts, among them SW1 SW_Push, SW10 SW_Push, SW100 SW_Push, SW101 SW_Push, SW102 SW_Push, SW103 SW_Push, SW104 SW_Push, SW105 SW_Push, SW11 SW_Push, SW12 SW_Push, SW13 SW_Push, SW14 SW_Push, SW15 SW_Push, SW16 SW_Push, SW17 SW_Push, SW18 SW_Push, SW19 SW_Push, SW2 SW_Push, SW20 SW_Push, SW21 SW_Push, SW22 SW_Push, SW23 SW_Push, SW24 SW_Push, SW25 SW_Push, SW26 SW_Push, SW27 SW_Push, SW28 SW_Push, SW29 SW_Push, SW3 SW_Push, SW30 SW_Push, SW31 SW_Push, SW32 SW_Push, SW33 SW_Push, SW34 SW_Push, SW35 SW_Push, SW36 SW_Push, SW37 SW_Push, SW38 SW_Push, SW39 SW_Push, SW4 SW_Push, SW40 SW_Push, SW41 SW_Push, SW42 SW_Push, SW43 SW_Push, SW44 SW_Push, SW45 SW_Push, SW46 SW_Push, SW47 SW_Push, SW48 SW_Push, SW49 SW_Push, SW5 SW_Push, SW50 SW_Push, SW51 SW_Push, SW52 SW_Push, SW53 SW_Push, SW54 SW_Push, SW55 SW_Push, SW56 SW_Push, SW57 SW_Push, SW58 SW_Push, SW59 SW_Push, SW6 SW_Push, SW60 SW_Push, SW61 SW_Push, SW62 SW_Push, SW63 SW_Push, SW64 SW_Push, SW65 SW_Push, SW66 SW_Push, SW67 SW_Push, SW68 SW_Push, SW69 SW_Push, SW7 SW_Push, SW70 SW_Push, SW71 SW_Push, SW72 SW_Push, SW73 SW_Push, SW74 SW_Push, SW75 SW_Push, SW76 SW_Push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

Commit message: did more work on traces and added capacitors and hotswappable switches
Parts:
- removed LED? (x100): SK6812MINI-E, LED_SMD:LED_SK6812MINI-E_3.2x2.8mm_P1.5mm_ReverseMount, symbol LED:SK6812MINI-E
- removed U3: MCP23017x-x-SP, Package_DIP:DIP-28_W7.62mm, symbol Interface_Expansion:MCP23017x-x-SP
- added R1, R2: 4.7k, Resistor_THT:R_Axial_DIN0207_L6.3mm_D2.5mm_P7.62mm_Horizontal, symbol Device:R
Connections:
- net +3V3: now also A1.36 (3V3), R1.2, R2.1; no longer A1.37 (3V3_EN)
- net COL10: now also A1.11 (GPIO8)
- net COL11: now also A1.12 (GPIO9)
- net COL12: now also A1.14 (GPIO10)
- net COL13: now also A1.15 (GPIO11)
- net COL14: now also A1.16 (GPIO12)
- net COL15: now also A1.17 (GPIO13)
- net COL16: now also A1.19 (GPIO14)
- net COL17: now also A1.20 (GPIO15)
- net COL18: now also A1.21 (GPIO16)
- net COL19: now also A1.22 (GPIO17)
- net COL20: now also A1.24 (GPIO18)
- net ROTA: now also A1.25 (GPIO19)
- net ROTB: now also A1.26 (GPIO20)
- net ROTBU: now also A1.27 (GPIO21)
- net SCL: now also R2.2
- net SDA: now also R1.1
- net DIN: now reaches A1.10 (GPIO7)
- net +5V: now reaches A1.40 (VBUS)
- net +5V: now also U1.2 (VCC)
- net INTB: no longer names the net of A1.9 (GPIO6)
- net VSYS: no longer names the net of A1.39 (VSYS)
- net VSYS: no longer U1.2 (VCC)
Other:
- added sheet RGB_LEDs (leds.kicad_sch)

Commit message: more journalling
Parts:
- D1, D10, D100, D101, D102, D103, D104, D105, D11, D12, D13, D14, D15, D16, D17, D18, D19, D2, D20, D21, D22, D23, D24, D25, D26, D27, D28, D29, D3, D30, D31, D32, D33, D34, D35, D36, D37, D38, D39, D4, D40, D41, D42, D43, D44, D45, D46, D47, D48, D49, D5, D50, D51, D52, D53, D54, D55, D56, D57, D58, D59, D6, D60, D61, D62, D63, D64, D65, D66, D67, D68, D69, D7, D70, D71, D72, D73, D74, D75, D76, D77, D78, D79, D8, D80, D81, D82, D83, D84, D85, D86, D87, D88, D89, D9, D90, D91, D92, D93, D94, D95, D96, D97, D98, D99: footprint Diode_THT:D_DO-35_SOD27_P7.62mm_Horizontal -> Diode_SMD:D_SOD-123F; KiLib_Generator (none) -> diode/THT
- R1, R2: KiLib_Generator (none) -> resistor/THT
- SW1, SW10, SW100, SW101, SW102, SW103, SW104, SW105, SW11, SW12, SW13, SW14, SW15, SW16, SW17, SW18, SW19, SW2, SW20, SW21, SW22, SW23, SW24, SW25, SW26, SW27, SW28, SW29, SW3, SW30, SW31, SW32, SW33, SW34, SW35, SW36, SW37, SW38, SW39, SW4, SW40, SW41, SW42, SW43, SW44, SW45, SW46, SW47, SW48, SW49, SW5, SW50, SW51, SW52, SW53, SW54, SW55, SW56, SW57, SW58, SW59, SW6, SW60, SW61, SW62, SW63, SW64, SW65, SW66, SW67, SW68, SW69, SW7, SW70, SW71, SW72, SW73, SW74, SW75, SW76, SW77, SW78, SW79, SW8, SW80, SW81, SW82, SW83, SW84, SW85, SW86, SW87, SW88, SW89, SW9, SW90, SW91, SW92, SW93, SW94, SW95, SW96, SW97, SW98, SW99: footprint PCM_marbastlib-mx:SW_MX_1u -> PCM_marbastlib-mx:SW_MX_HS_CPG151101S11_1u
- U2: KiLib_Generator (none) -> package/DIP/legacy
Connections:
- net +3V3: now also A1.37 (3V3_EN)
- net VSYS: now reaches A1.39 (VSYS)

Commit message: did more work and journaling
Connections:
- net COL0: now also A1.34 (GPIO28_ADC2); no longer U2.27 (GPA6)
- net COL1: now also A1.32 (GPIO27_ADC1); no longer U2.28 (GPA7)
- net COL10: now also A1.20 (GPIO15); no longer A1.11 (GPIO8)
- net COL11: now also U2.8 (GPB7); no longer A1.12 (GPIO9)
- net COL12: now also U2.7 (GPB6); no longer A1.14 (GPIO10)
- net COL13: now also U2.6 (GPB5); no longer A1.15 (GPIO11)
- net COL14: now also U2.5 (GPB4); no longer A1.16 (GPIO12)
- net COL15: now also U2.4 (GPB3); no longer A1.17 (GPIO13)
- net COL16: now also U2.3 (GPB2); no longer A1.19 (GPIO14)
- net COL17: now also U2.2 (GPB1); no longer A1.20 (GPIO15)
- net COL18: now also U2.1 (GPB0); no longer A1.21 (GPIO16)
- net COL19: now also U2.28 (GPA7); no longer A1.22 (GPIO17)
- net COL2: now also A1.31 (GPIO26_ADC0); no longer U2.1 (GPB0)
- net COL20: now also U2.27 (GPA6); no longer A1.24 (GPIO18)
- net COL3: now also A1.29 (GPIO22); no longer U2.2 (GPB1)
- net COL4: now also A1.27 (GPIO21); no longer U2.3 (GPB2)
- net COL5: now also A1.26 (GPIO20); no longer U2.4 (GPB3)
- net COL6: now also A1.25 (GPIO19); no longer U2.5 (GPB4)
- net COL7: now also A1.24 (GPIO18); no longer U2.6 (GPB5)
- net COL8: now also A1.22 (GPIO17); no longer U2.7 (GPB6)
- net COL9: now also A1.21 (GPIO16); no longer U2.8 (GPB7)
- net ROTA: now also A1.16 (GPIO12); no longer A1.25 (GPIO19)
- net ROTB: now also A1.17 (GPIO13); no longer A1.26 (GPIO20)
- net ROTBU: now also A1.19 (GPIO14); no longer A1.27 (GPIO21)
Changed lines of the file:
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@@
 	(wire
 		(pts
+			(xy 293.37 257.81) (xy 299.72 257.81)
+		)
+		(stroke
+			(width 0)
+			(type default)
+		)
+	)
+	(wire
+		(pts
 			(xy 120.65 97.79) (xy 135.89 97.79)
 		)
@@
 	(wire
 		(pts
-			(xy 241.3 250.19) (xy 247.65 250.19)
-		)
-		(stroke
-			(width 0)
-			(type default)
-		)
-	)
-	(wire
-		(pts
 			(xy 92.71 214.63) (xy 99.06 214.63)
 		)
@@
 	(wire
 		(pts
-			(xy 241.3 247.65) (xy 247.65 247.65)
+			(xy 293.37 242.57) (xy 299.72 242.57)
 		)
 		(stroke
@@
 	(wire
 		(pts
+			(xy 293.37 252.73) (xy 299.72 252.73)
+		)
+		(stroke
+			(width 0)
+			(type default)
+		)
+	)
+	(wire
+		(pts
 			(xy 240.03 237.49) (xy 247.65 237.49)
 		)
@@
 	(wire
 		(pts
-			(xy 241.3 245.11) (xy 247.65 245.11)
-		)
-		(stroke
-			(width 0)
-			(type default)
-		)
-	)
-	(wire
-		(pts
 			(xy 215.9 25.4) (xy 219.71 25.4)
 		)
@@
 	(wire
 		(pts
-			(xy 241.3 252.73) (xy 247.65 252.73)
-		)
-		(stroke
-			(width 0)
-			(type default)
-		)
-	)
-	(wire
-		(pts
 			(xy 149.86 63.5) (xy 151.13 63.5)
 		)
@@
 	(wire
 		(pts
+			(xy 293.37 255.27) (xy 299.72 255.27)
+		)
+		(stroke
+			(width 0)
+			(type default)
+		)
+	)
+	(wire
+		(pts
 			(xy 92.71 224.79) (xy 99.06 224.79)
 		)
@@
 		)
 	)
-	(label "COL4"
-		(at 92.71 227.33 0)
-		(effects
-			(font
-				(size 1.27 1.27)
-			)
-			(justify left bottom)
-		)
-	)
 	(label "ROW2"
 		(at 17.78 97.79 0)
@@
 		)
 	)
-	(label "COL5"
-		(at 92.71 229.87 0)
-		(effects
-			(font
-				(size 1.27 1.27)
-			)
-			(justify left bottom)
-		)
-	)
 	(label "SCL"
 		(at 369.57 60.96 0)
@@
 		)
 	)
-	(label "COL15"
-		(at 241.3 257.81 0)
-		(effects
-			(font
-				(size 1.27 1.27)
-			)
-			(justify left bottom)
-		)
-	)
-	(label "COL2"
-		(at 92.71 222.25 0)
-		(effects
-			(font
-				(size 1.27 1.27)
-			)
-			(justify left bottom)
-		)
-	)
-	(label "COL13"
-		(at 241.3 252.73 0)
-		(effects
-			(font
-				(size 1.27 1.27)
-			)
-			(justify left bottom)
-		)
-	)
 	(label "SDA"
 		(at 229.87 234.95 0)
@@
 		)
 	)
-	(label "ROTA"
-		(at 293.37 234.95 0)
+	(label "COL4"
+		(at 93.98 25.4 0)
 		(effects
 			(font
@@
 		)
 	)
-	(label "COL4"
-		(at 93.98 25.4 0)
+	(label "COL20"
+		(at 92.71 214.63 0)
 		(effects
 			(font
@@
 		)
 	)
-	(label "ROTBU"
-		(at 293.37 240.03 0)
+	(label "COL3"
+		(at 78.74 25.4 0)
 		(effects
 			(font
@@
 		)
 	)
-	(label "COL3"
-		(at 78.74 25.4 0)
+	(label "COL1"
+		(at 293.37 255.27 0)
 		(effects
 			(font
@@
 		)
 	)
-	(label "COL16"
-		(at 241.3 260.35 0)
+	(label "COL17"
+		(at 92.71 224.79 0)
 		(effects
 			(font
@@
 		)
 	)
-	(label "COL1"
-		(at 92.71 217.17 0)
+	(label "COL12"
+		(at 92.71 237.49 0)
 		(effects
 			(font
@@
 		)
 	)
-	(label "COL3"
-		(at 92.71 224.79 0)
+	(label "COL8"
+		(at 293.37 229.87 0)
 		(effects
 			(font
@@
 		)
 	)
+	(label "COL3"
+		(at 293.37 242.57 0)
+		(effects
+			(font
+				(size 1.27 1.27)
+			)
+			(justify left bottom)
+		)
+	)
 	(label "COL13"
 		(at 231.14 25.4 0)
@@
 		)
 	)
-	(label "COL8"
-		(at 92.71 237.49 0)
+	(label "COL9"
+		(at 293.37 227.33 0)
 		(effects
 			(font
@@
 		)
 	)
-	(label "COL11"
-		(at 241.3 247.65 0)
+	(label "COL0"
+		(at 293.37 257.81 0)
+		(effects
+			(font
+				(size 1.27 1.27)
+			)
+			(justify left bottom)
+		)
+	)
+	(label "COL5"
+		(at 293.37 237.49 0)
+		(effects
+			(font
+				(size 1.27 1.27)
+			)
+			(justify left bottom)
+		)
+	)
+	(label "COL6"
+		(at 293.37 234.95 0)
 		(effects
 			(font
@@
 		)
 	)
-	(label "COL11"
-		(at 200.66 25.4 0)
+	(label "ROTBU"
+		(at 241.3 260.35 0)
 		(effects
 			(font
@@
 		)
 	)
-	(label "COL19"
-		(at 293.37 229.87 0)
+	(label "COL11"
+		(at 200.66 25.4 0)
 		(effects
 			(font
@@
 		)
 	)
+	(label "COL15"
+		(at 92.71 229.87 0)
+		(effects
+			(font
+				(size 1.27 1.27)
+			)
+			(justify left bottom)
+		)
+	)
+	(label "COL4"
+		(at 293.37 240.03 0)
+		(effects
+			(font
+				(size 1.27 1.27)
+			)
+			(justify left bottom)
+		)
+	)
+	(label "COL10"
+		(at 241.3 262.89 0)
+		(effects
+			(font
+				(size 1.27 1.27)
+			)
+			(justify left bottom)
+		)
+	)
+	(label "COL16"
+		(at 92.71 227.33 0)
+		(effects
+			(font
+				(size 1.27 1.27)
+			)
+			(justify left bottom)
+		)
+	)
 	(label "ROW5"
 		(at 17.78 173.99 0)
@@
 		)
 	)
-	(label "COL9"
-		(at 92.71 240.03 0)
+	(label "COL14"
+		(at 92.71 232.41 0)
 		(effects
 			(font
@@
 		)
 	)
-	(label "COL20"
-		(at 293.37 232.41 0)
-		(effects
-			(font
-				(size 1.27 1.27)
-			)
-			(justify left bottom)
-		)
-	)
 	(label "COL8"
 		(at 154.94 25.4 0)
@@
 		)
 	)
-	(label "COL6"
-		(at 92.71 232.41 0)
+	(label "COL13"
+		(at 92.71 234.95 0)
 		(effects
 			(font
@@
 		)
 	)
-	(label "COL0"
-		(at 92.71 214.63 0)
+	(label "ROTA"
+		(at 241.3 255.27 0)
+		(effects
+			(font
+				(size 1.27 1.27)
+			)
+			(justify left bottom)
+		)
+	)
+	(label "COL11"
+		(at 92.71 240.03 0)
 		(effects
 			(font
@@
 		)
 	)
-	(label "COL12"
-		(at 241.3 250.19 0)
+	(label "COL19"
+		(at 92.71 217.17 0)
 		(effects
 			(font
@@
 		)
 	)
-	(label "COL6"
-		(at 124.46 25.4 0)
+	(label "ROTB"
+		(at 241.3715 257.81 0)
 		(effects
 			(font
@@
 		)
 	)
-	(label "COL17"
-		(at 241.3 262.89 0)
+	(label "COL6"
+		(at 124.46 25.4 0)
 		(effects
 			(font
@@
 		)
 	)
-	(label "ROTA"
-		(at 370.84 34.29 0)
-		(effects
-			(font
-				(size 1.27 1.27)
-			)
-			(justify left bottom)
-		)
-	)
-	(label "ROW1"
-		(at 92.71 201.93 0)
+	(label "COL2"
+		(at 293.37 252.73 0)
 		(effects
 			(font
@@
 		)
 	)
-	(label "COL10"
-		(at 241.3 245.11 0)
+	(label "ROTA"
+		(at 370.84 34.29 0)
 		(effects
 			(font
@@
 		)
 	)
-	(label "COL7"
-		(at 92.71 234.95 0)
+	(label "ROW1"
+		(at 92.71 201.93 0)
 		(effects
 			(font
@@
 		)
 	)
-	(label "ROTB"
-		(at 293.37 237.49 0)
+	(label "COL18"
+		(at 92.71 222.25 0)
 		(effects
 			(font
@@
 		)
 	)
-	(label "COL14"
-		(at 241.3 255.27 0)
+	(label "COL7"
+		(at 293.37 232.41 0)
 		(effects
 			(font
@@
 		(effects
 			(font
-				(size 1.27 1.27)
-			)
-			(justify left bottom)
-		)
-	)
-	(label "COL18"
-		(at 293.37 227.33 0)
-		(effects
-			(font

Commit message: did more routing
Connections:
- net DIN: now also A1.19 (GPIO14); no longer A1.10 (GPIO7)
- net GND: now also ROT_SW1.MP
- net ROTA: now also A1.15 (GPIO11); no longer A1.16 (GPIO12)
- net ROTB: now also A1.16 (GPIO12); no longer A1.17 (GPIO13)
- net ROTBU: now also A1.17 (GPIO13); no longer A1.19 (GPIO14)
Changed lines of the file:
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@@
 	(wire
 		(pts
+			(xy 241.3 255.27) (xy 247.65 255.27)
+		)
+		(stroke
+			(width 0)
+			(type default)
+		)
+	)
+	(wire
+		(pts
 			(xy 120.65 173.99) (xy 135.89 173.99)
 		)
@@
 	(wire
 		(pts
+			(xy 241.3 252.73) (xy 247.65 252.73)
+		)
+		(stroke
+			(width 0)
+			(type default)
+		)
+	)
+	(wire
+		(pts
 			(xy 180.34 88.9) (xy 181.61 88.9)
 		)
@@
 	(wire
 		(pts
-			(xy 241.3 242.57) (xy 247.65 242.57)
-		)
-		(stroke
-			(width 0)
-			(type default)
-		)
-	)
-	(wire
-		(pts
 			(xy 369.57 66.04) (xy 373.38 66.04)
 		)
@@
 	(wire
 		(pts
+			(xy 241.3 257.81) (xy 247.65 257.81)
+		)
+		(stroke
+			(width 0)
+			(type default)
+		)
+	)
+	(wire
+		(pts
 			(xy 307.34 63.5) (xy 307.34 88.9)
 		)
@@
 	(wire
 		(pts
-			(xy 246.38 88.9) (xy 246.38 165.1)
+			(xy 241.3 260.35) (xy 247.65 260.35)
 		)
 		(stroke
@@
 	(wire
 		(pts
-			(xy 43.18 114.3) (xy 44.45 114.3)
+			(xy 246.38 88.9) (xy 246.38 165.1)
 		)
 		(stroke
@@
 	(wire
 		(pts
-			(xy 227.33 46.99) (xy 257.81 46.99)
+			(xy 43.18 114.3) (xy 44.45 114.3)
 		)
 		(stroke
@@
 	(wire
 		(pts
-			(xy 17.78 72.39) (xy 44.45 72.39)
+			(xy 227.33 46.99) (xy 257.81 46.99)
 		)
 		(stroke
@@
 	(wire
 		(pts
-			(xy 48.26 114.3) (xy 48.26 139.7)
+			(xy 17.78 72.39) (xy 44.45 72.39)
 		)
 		(stroke
@@
 	(wire
 		(pts
-			(xy 120.65 38.1) (xy 120.65 39.37)
+			(xy 48.26 114.3) (xy 48.26 139.7)
 		)
 		(stroke
@@
 	(wire
 		(pts
-			(xy 241.3 260.35) (xy 247.65 260.35)
+			(xy 120.65 38.1) (xy 120.65 39.37)
 		)
 		(stroke
@@
 	(wire
 		(pts
-			(xy 241.3 255.27) (xy 247.65 255.27)
-		)
-		(stroke
-			(width 0)
-			(type default)
-		)
-	)
-	(wire
-		(pts
 			(xy 90.17 165.1) (xy 90.17 166.37)
 		)
@@
 	(wire
 		(pts
-			(xy 241.3 257.81) (xy 247.65 257.81)
-		)
-		(stroke
-			(width 0)
-			(type default)
-		)
-	)
-	(wire
-		(pts
 			(xy 92.71 222.25) (xy 99.06 222.25)
 		)
@@
 		)
 	)
+	(label "ROTBU"
+		(at 241.3 257.81 0)
+		(effects
+			(font
+				(size 1.27 1.27)
+			)
+			(justify left bottom)
+		)
+	)
 	(label "COL4"
 		(at 93.98 25.4 0)
@@
 		)
 	)
+	(label "ROTB"
+		(at 241.3715 255.27 0)
+		(effects
+			(font
+				(size 1.27 1.27)
+			)
+			(justify left bottom)
+		)
+	)
 	(label "COL3"
 		(at 78.74 25.4 0)
@@
 		)
 	)
-	(label "ROTBU"
-		(at 241.3 260.35 0)
-		(effects
-			(font
-				(size 1.27 1.27)
-			)
-			(justify left bottom)
-		)
-	)
 	(label "COL11"
 		(at 200.66 25.4 0)
@@
 		)
 	)
-	(label "ROTA"
-		(at 241.3 255.27 0)
-		(effects
-			(font
-				(size 1.27 1.27)
-			)
-			(justify left bottom)
-		)
-	)
 	(label "COL11"
 		(at 92.71 240.03 0)
@@
 		)
 	)
-	(label "ROTB"
-		(at 241.3715 257.81 0)
-		(effects
-			(font
-				(size 1.27 1.27)
-			)
-			(justify left bottom)
-		)
-	)
 	(label "COL6"
 		(at 124.46 25.4 0)
@@
 		)
 	)
+	(label "ROTA"
+		(at 241.3 252.73 0)
+		(effects
+			(font
+				(size 1.27 1.27)
+			)
+			(justify left bottom)
+		)
+	)
 	(label "COL0"
 		(at 33.02 25.4 0)
@@
 	(global_label "DIN"
 		(shape input)
-		(at 241.3 242.57 180)
+		(at 241.3 260.35 180)
 		(fields_autoplaced yes)
 		(effects
@@
 		)
 		(property "Intersheetrefs" "${INTERSHEET_REFS}"
-			(at 235.1095 242.57 0)
+			(at 235.1095 260.35 0)
 			(hide yes)
 			(show_name no)
@@
 					(unit 1)
 				)
+			)
+		)
+	)
+	(symbol
+		(lib_id "power:GND")
+		(at 383.54 44.45 90)
+		(unit 1)
+		(body_style 1)
+		(exclude_from_sim no)
+		(in_bom yes)
+		(on_board yes)
+		(in_pos_files yes)
+		(dnp no)
+		(fields_autoplaced yes)
+		(property "Reference" "#PWR0222"
+			(at 389.89 44.45 0)
+			(hide yes)
+			(show_name no)
+			(do_not_autoplace no)
+			(effects
+				(font
+					(size 1.27 1.27)
+				)
+			)
+		)
+		(property "Value" "GND"
+			(at 387.35 44.4499 90)
+			(show_name no)
+			(do_not_autoplace no)
+			(effects
+				(font
+					(size 1.27 1.27)
+				)
+				(justify right)
+			)
+		)
+		(property "Footprint" ""
+			(at 383.54 44.45 0)
+			(hide yes)
+			(show_name no)
+			(do_not_autoplace no)
+			(effects
+				(font
+					(size 1.27 1.27)
+				)
+			)
+		)
+		(property "Datasheet" ""
+			(at 383.54 44.45 0)
+			(hide yes)
+			(show_name no)
+			(do_not_autoplace no)
+			(effects
+				(font
+					(size 1.27 1.27)
+				)
+			)
+		)
+		(property "Description" "Power symbol creates a global label with name \"GND\" , ground"
+			(at 383.54 44.45 0)
+			(hide yes)
+			(show_name no)
+			(do_not_autoplace no)
+			(effects
+				(font
+					(size 1.27 1.27)
+				)
+			)
+		)
+		(pin "1"
+		)
+		(instances
+			(project "keeb"
+				(path "/a754da10-386a-4d11-8b4c-7b14c49d2f59"
+					(reference "#PWR0222")
+					(unit 1)
+				)

Commit message: PCB DESIGN DONE!!!!
Connections:
- net ROTA: now also A1.16 (GPIO12); no longer A1.15 (GPIO11)
- net ROTB: now also A1.17 (GPIO13); no longer A1.16 (GPIO12)
- net ROTBU: now also A1.15 (GPIO11); no longer A1.17 (GPIO13)
Changed lines of the file:
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@@
-		)
-	)
-	(label "ROTBU"
-		(at 241.3 257.81 0)
-		(effects
-			(font
-				(size 1.27 1.27)
-			)
-			(justify left bottom)
 		)
 	)
@@
 		)
 	)
-	(label "ROTB"
-		(at 241.3715 255.27 0)
-		(effects
-			(font
-				(size 1.27 1.27)
-			)
-			(justify left bottom)
-		)
-	)
 	(label "COL3"
 		(at 78.74 25.4 0)
@@
 		)
 	)
+	(label "ROTB"
+		(at 241.3 257.81 0)
+		(effects
+			(font
+				(size 1.27 1.27)
+			)
+			(justify left bottom)
+		)
+	)
 	(label "COL10"
 		(at 241.3 262.89 0)
@@
 		)
 	)
+	(label "ROTA"
+		(at 241.3 255.27 0)
+		(effects
+			(font
+				(size 1.27 1.27)
+			)
+			(justify left bottom)
+		)
+	)
 	(label "COL8"
 		(at 154.94 25.4 0)
@@
 		)
 	)
+	(label "ROTBU"
+		(at 241.3 252.73 0)
+		(effects
+			(font
+				(size 1.27 1.27)
+			)
+			(justify left bottom)
+		)
+	)
 	(label "COL6"
 		(at 124.46 25.4 0)
@@
 		(effects
 			(font
-				(size 1.27 1.27)
-			)
-			(justify left bottom)
-		)
-	)
-	(label "ROTA"
-		(at 241.3 252.73 0)
-		(effects
-			(font

Commit message: i hate fusion
Parts:
- S1, S2, S3, S4, S5, S6: now left out of the parts list
Changed lines of the file:
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@@
 		(body_style 1)
 		(exclude_from_sim no)
-		(in_bom yes)
+		(in_bom no)
 		(on_board yes)
 		(in_pos_files yes)
@@
 		(body_style 1)
 		(exclude_from_sim no)
-		(in_bom yes)
+		(in_bom no)
 		(on_board yes)
 		(in_pos_files yes)
@@
 		(body_style 1)
 		(exclude_from_sim no)
-		(in_bom yes)
+		(in_bom no)
 		(on_board yes)
 		(in_pos_files yes)
@@
 		(body_style 1)
 		(exclude_from_sim no)
-		(in_bom yes)
+		(in_bom no)
 		(on_board yes)
 		(in_pos_files yes)
@@
 		(body_style 1)
 		(exclude_from_sim no)
-		(in_bom yes)
+		(in_bom no)
 		(on_board yes)
 		(in_pos_files yes)
@@
 		(body_style 1)
 		(exclude_from_sim no)
-		(in_bom yes)
+		(in_bom no)
 		(on_board yes)
 		(in_pos_files yes)
