File: _autosave-keeb.kicad_sch (KiCad schematic)
At the start: 321 parts, among them SW1 SW_Push, SW10 SW_Push, SW100 SW_Push, SW101 SW_Push, SW102 SW_Push, SW103 SW_Push, SW104 SW_Push, SW105 SW_Push, SW11 SW_Push, SW12 SW_Push, SW13 SW_Push, SW14 SW_Push, SW15 SW_Push, SW16 SW_Push, SW17 SW_Push, SW18 SW_Push, SW19 SW_Push, SW2 SW_Push, SW20 SW_Push, SW21 SW_Push, SW22 SW_Push, SW23 SW_Push, SW24 SW_Push, SW25 SW_Push, SW26 SW_Push, SW27 SW_Push, SW28 SW_Push, SW29 SW_Push, SW3 SW_Push, SW30 SW_Push, SW31 SW_Push, SW32 SW_Push, SW33 SW_Push, SW34 SW_Push, SW35 SW_Push, SW36 SW_Push, SW37 SW_Push, SW38 SW_Push, SW39 SW_Push, SW4 SW_Push, SW40 SW_Push, SW41 SW_Push, SW42 SW_Push, SW43 SW_Push, SW44 SW_Push, SW45 SW_Push, SW46 SW_Push, SW47 SW_Push, SW48 SW_Push, SW49 SW_Push, SW5 SW_Push, SW50 SW_Push, SW51 SW_Push, SW52 SW_Push, SW53 SW_Push, SW54 SW_Push, SW55 SW_Push, SW56 SW_Push, SW57 SW_Push, SW58 SW_Push, SW59 SW_Push, SW6 SW_Push, SW60 SW_Push, SW61 SW_Push, SW62 SW_Push, SW63 SW_Push, SW64 SW_Push, SW65 SW_Push, SW66 SW_Push, SW67 SW_Push, SW68 SW_Push, SW69 SW_Push, SW7 SW_Push, SW70 SW_Push, SW71 SW_Push, SW72 SW_Push, SW73 SW_Push, SW74 SW_Push, SW75 SW_Push, SW76 SW_Push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

Commit message: been 4 hours of CHANGING EVERYTHING AAAAAAAAAAAAAAAAAAAAAAAAAAAA
Parts:
- removed LED? (x80): SK6812MINI-E, LED_SMD:LED_SK6812MINI-E_3.2x2.8mm_P1.5mm_ReverseMount, symbol LED:SK6812MINI-E
- removed U3: MCP23017x-x-SP, Package_DIP:DIP-28_W7.62mm, symbol Interface_Expansion:MCP23017x-x-SP
- added LED100, LED101, LED102, LED103, LED104, LED105, LED21, LED22, LED23, LED24, LED25, LED26, LED27, LED28, LED29, LED30, LED31, LED32, LED33, LED34, LED35, LED36, LED37, LED38, LED39, LED40, LED41, LED42, LED43, LED44, LED45, LED46, LED47, LED48, LED49, LED50, LED51, LED52, LED53, LED54, LED55, LED56, LED57, LED58, LED59, LED60, LED61, LED62, LED63, LED64, LED65, LED66, LED67, LED68, LED69, LED70, LED71, LED72, LED73, LED74, LED75, LED76, LED77, LED78, LED79, LED80, LED81, LED82, LED83, LED84, LED85, LED86, LED87, LED88, LED89, LED90, LED91, LED92, LED93, LED94, LED95, LED96, LED97, LED98, LED99: SK6812MINI-E, LED_SMD:LED_SK6812MINI-E_3.2x2.8mm_P1.5mm_ReverseMount, symbol LED:SK6812MINI-E
- added R1: 300, Resistor_THT:R_Axial_DIN0207_L6.3mm_D2.5mm_P7.62mm_Horizontal, symbol Device:R
- added R2, R3: 4.7k, Resistor_THT:R_Axial_DIN0207_L6.3mm_D2.5mm_P7.62mm_Horizontal, symbol Device:R
- gave numbers to parts that had none: 20
Connections:
- net +3V3: now also R2.2, R3.1
- net COL10: now also A1.11 (GPIO8)
- net COL11: now also A1.12 (GPIO9)
- net COL12: now also A1.14 (GPIO10)
- net COL13: now also A1.15 (GPIO11)
- net COL14: now also A1.16 (GPIO12)
- net COL15: now also A1.17 (GPIO13)
- net COL16: now also A1.19 (GPIO14)
- net COL17: now also A1.20 (GPIO15)
- net COL18: now also A1.21 (GPIO16)
- net COL19: now also A1.22 (GPIO17)
- net COL20: now also A1.24 (GPIO18)
- net GND: now also LED1.1 (VSS), LED10.1 (VSS), LED11.1 (VSS), LED12.1 (VSS), LED13.1 (VSS), LED14.1 (VSS), LED15.1 (VSS), LED16.1 (VSS), LED17.1 (VSS), LED18.1 (VSS), LED19.1 (VSS), LED2.1 (VSS), LED20.1 (VSS), LED3.1 (VSS), LED4.1 (VSS), LED5.1 (VSS), LED6.1 (VSS), LED7.1 (VSS), LED8.1 (VSS), LED9.1 (VSS), LED101.1 (VSS), LED102.1 (VSS), LED103.1 (VSS), LED104.1 (VSS), LED105.1 (VSS), LED21.1 (VSS), LED22.1 (VSS), LED23.1 (VSS), LED24.1 (VSS), LED25.1 (VSS), LED26.1 (VSS), LED27.1 (VSS), LED28.1 (VSS), LED29.1 (VSS), LED30.1 (VSS), LED31.1 (VSS), LED32.1 (VSS), LED33.1 (VSS), LED34.1 (VSS), LED35.1 (VSS), LED36.1 (VSS), LED37.1 (VSS), LED38.1 (VSS), LED39.1 (VSS), LED40.1 (VSS), LED41.1 (VSS), LED42.1 (VSS), LED43.1 (VSS), LED44.1 (VSS), LED45.1 (VSS), LED46.1 (VSS), LED47.1 (VSS), LED48.1 (VSS), LED49.1 (VSS), LED50.1 (VSS), LED51.1 (VSS), LED52.1 (VSS), LED53.1 (VSS), LED54.1 (VSS), LED55.1 (VSS), LED56.1 (VSS), LED57.1 (VSS), LED58.1 (VSS), LED59.1 (VSS), LED60.1 (VSS), LED61.1 (VSS), LED62.1 (VSS), LED63.1 (VSS), LED64.1 (VSS), LED65.1 (VSS), LED66.1 (VSS), LED67.1 (VSS), LED68.1 (VSS), LED69.1 (VSS), LED70.1 (VSS), LED71.1 (VSS), LED72.1 (VSS), LED73.1 (VSS), LED74.1 (VSS), LED75.1 (VSS), LED76.1 (VSS), LED77.1 (VSS), LED78.1 (VSS), LED79.1 (VSS), LED80.1 (VSS), LED81.1 (VSS), LED82.1 (VSS), LED83.1 (VSS), LED84.1 (VSS), LED85.1 (VSS), LED86.1 (VSS), LED87.1 (VSS), LED88.1 (VSS), LED89.1 (VSS), LED90.1 (VSS)
- net ROTA: now also A1.25 (GPIO19)
- net ROTB: now also A1.26 (GPIO20)
- net ROTBU: now also A1.27 (GPIO21)
- net SCL: now also R3.2
- net SDA: now also R2.1
- net VSYS: now also LED1.3 (VDD), LED10.3 (VDD), LED11.3 (VDD), LED12.3 (VDD), LED13.3 (VDD), LED14.3 (VDD), LED15.3 (VDD), LED16.3 (VDD), LED17.3 (VDD), LED18.3 (VDD), LED19.3 (VDD), LED2.3 (VDD), LED20.3 (VDD), LED3.3 (VDD), LED4.3 (VDD), LED5.3 (VDD), LED6.3 (VDD), LED7.3 (VDD), LED8.3 (VDD), LED9.3 (VDD), LED100.3 (VDD), LED101.3 (VDD), LED102.3 (VDD), LED103.3 (VDD), LED104.3 (VDD), LED105.3 (VDD), LED21.3 (VDD), LED22.3 (VDD), LED23.3 (VDD), LED24.3 (VDD), LED25.3 (VDD), LED26.3 (VDD), LED27.3 (VDD), LED28.3 (VDD), LED29.3 (VDD), LED30.3 (VDD), LED31.3 (VDD), LED32.3 (VDD), LED33.3 (VDD), LED34.3 (VDD), LED35.3 (VDD), LED36.3 (VDD), LED37.3 (VDD), LED38.3 (VDD), LED39.3 (VDD), LED40.3 (VDD), LED41.3 (VDD), LED42.3 (VDD), LED43.3 (VDD), LED44.3 (VDD), LED45.3 (VDD), LED46.3 (VDD), LED47.3 (VDD), LED48.3 (VDD), LED49.3 (VDD), LED50.3 (VDD), LED51.3 (VDD), LED52.3 (VDD), LED53.3 (VDD), LED54.3 (VDD), LED55.3 (VDD), LED56.3 (VDD), LED57.3 (VDD), LED58.3 (VDD), LED59.3 (VDD), LED60.3 (VDD), LED61.3 (VDD), LED62.3 (VDD), LED63.3 (VDD), LED64.3 (VDD), LED65.3 (VDD), LED66.3 (VDD), LED67.3 (VDD), LED68.3 (VDD), LED69.3 (VDD), LED70.3 (VDD), LED71.3 (VDD), LED72.3 (VDD), LED73.3 (VDD), LED74.3 (VDD), LED75.3 (VDD), LED76.3 (VDD), LED77.3 (VDD), LED78.3 (VDD), LED79.3 (VDD), LED80.3 (VDD), LED81.3 (VDD), LED82.3 (VDD), LED83.3 (VDD), LED84.3 (VDD), LED85.3 (VDD), LED86.3 (VDD), LED87.3 (VDD), LED88.3 (VDD), LED89.3 (VDD), LED90.3 (VDD), LED91.3 (VDD), LED92.3 (VDD), LED93.3 (VDD), LED94.3 (VDD), LED95.3 (VDD), LED96.3 (VDD), LED97.3 (VDD), LED98.3 (VDD), LED99.3 (VDD)
- net at LED1.2 (DIN): now also R1.2
- net DIN: now reaches A1.10 (GPIO7)
- net DIN: now also R1.1
- net at LED20.4 (DOUT): now also LED21.2 (DIN)
- net at LED10.4 (DOUT): now also LED11.2 (DIN)
- net INTB: no longer names the net of A1.9 (GPIO6)
- new net: LED68.4 (DOUT), LED69.2 (DIN)
- new net: LED69.4 (DOUT), LED70.2 (DIN)
- new net: LED97.4 (DOUT), LED98.2 (DIN)
- new net: LED98.4 (DOUT), LED99.2 (DIN)
- new net: LED34.4 (DOUT), LED35.2 (DIN)
- new net: LED35.4 (DOUT), LED36.2 (DIN)
- new net: LED78.4 (DOUT), LED79.2 (DIN)
- new net: LED79.4 (DOUT), LED80.2 (DIN)
- new net: LED90.4 (DOUT), LED91.2 (DIN)
- new net: LED91.4 (DOUT), LED92.2 (DIN)
- new net: LED80.4 (DOUT), LED81.2 (DIN)
- new net: LED42.4 (DOUT), LED43.2 (DIN)
- new net: LED43.4 (DOUT), LED44.2 (DIN)
- new net: LED82.4 (DOUT), LED83.2 (DIN)
- new net: LED83.4 (DOUT), LED84.2 (DIN)
- new net: LED66.4 (DOUT), LED67.2 (DIN)
- new net: LED67.4 (DOUT), LED68.2 (DIN)
- new net: LED81.4 (DOUT), LED82.2 (DIN)
- new net: LED27.4 (DOUT), LED28.2 (DIN)
- new net: LED28.4 (DOUT), LED29.2 (DIN)
- new net: LED54.4 (DOUT), LED55.2 (DIN)
- new net: LED55.4 (DOUT), LED56.2 (DIN)
- new net: LED70.4 (DOUT), LED71.2 (DIN)
- new net: LED104.4 (DOUT), LED105.2 (DIN)
- new net: LED57.4 (DOUT), LED58.2 (DIN)
- new net: LED58.4 (DOUT), LED59.2 (DIN)
- new net: LED62.4 (DOUT), LED63.2 (DIN)
- new net: LED63.4 (DOUT), LED64.2 (DIN)
- new net: LED101.4 (DOUT), LED102.2 (DIN)
- new net: LED102.4 (DOUT), LED103.2 (DIN)
- new net: LED56.4 (DOUT), LED57.2 (DIN)
- new net: LED71.4 (DOUT), LED72.2 (DIN)
- new net: LED39.4 (DOUT), LED40.2 (DIN)
- new net: LED40.4 (DOUT), LED41.2 (DIN)
- new net: LED103.4 (DOUT), LED104.2 (DIN)
- new net: LED21.4 (DOUT), LED22.2 (DIN)
- new net: LED25.4 (DOUT), LED26.2 (DIN)
- new net: LED26.4 (DOUT), LED27.2 (DIN)
- new net: LED96.4 (DOUT), LED97.2 (DIN)
- new net: LED30.4 (DOUT), LED31.2 (DIN)
- new net: LED31.4 (DOUT), LED32.2 (DIN)
- new net: LED89.4 (DOUT), LED90.2 (DIN)
- new net: LED65.4 (DOUT), LED66.2 (DIN)
- new net: LED92.4 (DOUT), LED93.2 (DIN)
- new net: LED93.4 (DOUT), LED94.2 (DIN)
- new net: LED76.4 (DOUT), LED77.2 (DIN)
- new net: LED77.4 (DOUT), LED78.2 (DIN)
- new net: LED38.4 (DOUT), LED39.2 (DIN)
- new net: LED72.4 (DOUT), LED73.2 (DIN)
- new net: LED73.4 (DOUT), LED74.2 (DIN)
- new net: LED41.4 (DOUT), LED42.2 (DIN)
- new net: LED74.4 (DOUT), LED75.2 (DIN)
- new net: LED46.4 (DOUT), LED47.2 (DIN)
- new net: LED47.4 (DOUT), LED48.2 (DIN)
- new net: LED48.4 (DOUT), LED49.2 (DIN)
- new net: LED49.4 (DOUT), LED50.2 (DIN)
- new net: LED59.4 (DOUT), LED60.2 (DIN)
- new net: LED60.4 (DOUT), LED61.2 (DIN)
- new net: LED52.4 (DOUT), LED53.2 (DIN)
- new net: LED53.4 (DOUT), LED54.2 (DIN)
- new net: LED100.2 (DIN), LED99.4 (DOUT)
- new net: LED36.4 (DOUT), LED37.2 (DIN)
- new net: LED51.4 (DOUT), LED52.2 (DIN)
- new net: LED100.4 (DOUT), LED101.2 (DIN)
- new net: LED29.4 (DOUT), LED30.2 (DIN)
- new net: LED87.4 (DOUT), LED88.2 (DIN)
- new net: LED88.4 (DOUT), LED89.2 (DIN)
- new net: LED23.4 (DOUT), LED24.2 (DIN)
- new net: LED24.4 (DOUT), LED25.2 (DIN)
- new net: LED22.4 (DOUT), LED23.2 (DIN)
- new net: LED94.4 (DOUT), LED95.2 (DIN)
- new net: LED61.4 (DOUT), LED62.2 (DIN)
- new net: LED64.4 (DOUT), LED65.2 (DIN)
- new net: LED75.4 (DOUT), LED76.2 (DIN)
- new net: LED84.4 (DOUT), LED85.2 (DIN)
- new net: LED50.4 (DOUT), LED51.2 (DIN)
- new net: LED95.4 (DOUT), LED96.2 (DIN)
- new net: LED33.4 (DOUT), LED34.2 (DIN)
- new net: LED86.4 (DOUT), LED87.2 (DIN)
- new net: LED37.4 (DOUT), LED38.2 (DIN)
- new net: LED44.4 (DOUT), LED45.2 (DIN)
- new net: LED32.4 (DOUT), LED33.2 (DIN)
- new net: LED45.4 (DOUT), LED46.2 (DIN)
- new net: LED85.4 (DOUT), LED86.2 (DIN)
Other:
- moved on the sheet: LED11, LED12, LED13, LED14, LED15, LED16, LED17, LED18, LED19, LED20

Commit message: did some more journalling
Parts:
- removed LED1, LED10, LED100, LED101, LED102, LED103, LED104, LED105, LED11, LED12, LED13, LED14, LED15, LED16, LED17, LED18, LED19, LED2, LED20, LED21, LED22, LED23, LED24, LED25, LED26, LED27, LED28, LED29, LED3, LED30, LED31, LED32, LED33, LED34, LED35, LED36, LED37, LED38, LED39, LED4, LED40, LED41, LED42, LED43, LED44, LED45, LED46, LED47, LED48, LED49, LED5, LED50, LED51, LED52, LED53, LED54, LED55, LED56, LED57, LED58, LED59, LED6, LED60, LED61, LED62, LED63, LED64, LED65, LED66, LED67, LED68, LED69, LED7, LED70, LED71, LED72, LED73, LED74, LED75, LED76, LED77, LED78, LED79, LED8, LED80, LED81, LED82, LED83, LED84, LED85, LED86, LED87, LED88, LED89, LED9, LED90, LED91, LED92, LED93, LED94, LED95, LED96, LED97, LED98, LED99: SK6812MINI-E, LED_SMD:LED_SK6812MINI-E_3.2x2.8mm_P1.5mm_ReverseMount, symbol LED:SK6812MINI-E
- removed R1: 300, Resistor_THT:R_Axial_DIN0207_L6.3mm_D2.5mm_P7.62mm_Horizontal, symbol Device:R
Connections:
- net +3V3: now also A1.36 (3V3); no longer A1.37 (3V3_EN)
- net +5V: now reaches A1.40 (VBUS)
- net +5V: now also U1.2 (VCC)
- net VSYS: no longer names the net of A1.39 (VSYS)
- net VSYS: no longer U1.2 (VCC)
Other:
- added sheet RGB_LEDs (leds.kicad_sch)

Commit message: did more work on traces and added capacitors and hotswappable switches
Parts:
- D1, D10, D100, D101, D102, D103, D104, D105, D11, D12, D13, D14, D15, D16, D17, D18, D19, D2, D20, D21, D22, D23, D24, D25, D26, D27, D28, D29, D3, D30, D31, D32, D33, D34, D35, D36, D37, D38, D39, D4, D40, D41, D42, D43, D44, D45, D46, D47, D48, D49, D5, D50, D51, D52, D53, D54, D55, D56, D57, D58, D59, D6, D60, D61, D62, D63, D64, D65, D66, D67, D68, D69, D7, D70, D71, D72, D73, D74, D75, D76, D77, D78, D79, D8, D80, D81, D82, D83, D84, D85, D86, D87, D88, D89, D9, D90, D91, D92, D93, D94, D95, D96, D97, D98, D99: footprint Diode_THT:D_DO-35_SOD27_P7.62mm_Horizontal -> Diode_SMD:D_SOD-123F; KiLib_Generator (none) -> diode/THT
- R1: renamed from R2; KiLib_Generator (none) -> resistor/THT
- R2: renamed from R3; KiLib_Generator (none) -> resistor/THT
- SW1, SW10, SW100, SW101, SW102, SW103, SW104, SW105, SW11, SW12, SW13, SW14, SW15, SW16, SW17, SW18, SW19, SW2, SW20, SW21, SW22, SW23, SW24, SW25, SW26, SW27, SW28, SW29, SW3, SW30, SW31, SW32, SW33, SW34, SW35, SW36, SW37, SW38, SW39, SW4, SW40, SW41, SW42, SW43, SW44, SW45, SW46, SW47, SW48, SW49, SW5, SW50, SW51, SW52, SW53, SW54, SW55, SW56, SW57, SW58, SW59, SW6, SW60, SW61, SW62, SW63, SW64, SW65, SW66, SW67, SW68, SW69, SW7, SW70, SW71, SW72, SW73, SW74, SW75, SW76, SW77, SW78, SW79, SW8, SW80, SW81, SW82, SW83, SW84, SW85, SW86, SW87, SW88, SW89, SW9, SW90, SW91, SW92, SW93, SW94, SW95, SW96, SW97, SW98, SW99: footprint PCM_marbastlib-mx:SW_MX_1u -> PCM_marbastlib-mx:SW_MX_HS_CPG151101S11_1u
- U2: KiLib_Generator (none) -> package/DIP/legacy
Connections:
- net +3V3: now also A1.37 (3V3_EN)
- net VSYS: now reaches A1.39 (VSYS)
