File: _autosave-keeb.kicad_pcb (KiCad board)
At the start: 2 copper layers, 3.6 x 3.2 mm, 433 parts, among them SW1 SW_Push, SW10 SW_Push, SW100 SW_Push, SW101 SW_Push, SW102 SW_Push, SW103 SW_Push, SW104 SW_Push, SW105 SW_Push, SW11 SW_Push, SW12 SW_Push, SW13 SW_Push, SW14 SW_Push, SW15 SW_Push, SW16 SW_Push, SW17 SW_Push, SW18 SW_Push, SW19 SW_Push, SW2 SW_Push, SW20 SW_Push, SW21 SW_Push, SW22 SW_Push, SW23 SW_Push, SW24 SW_Push, SW25 SW_Push, SW26 SW_Push, SW27 SW_Push, SW28 SW_Push, SW29 SW_Push, SW3 SW_Push, SW30 SW_Push, SW31 SW_Push, SW32 SW_Push, SW33 SW_Push, SW34 SW_Push, SW35 SW_Push, SW36 SW_Push, SW37 SW_Push, SW38 SW_Push, SW39 SW_Push, SW4 SW_Push, SW40 SW_Push, SW41 SW_Push, SW42 SW_Push, SW43 SW_Push, SW44 SW_Push, SW45 SW_Push, SW46 SW_Push, SW47 SW_Push, SW48 SW_Push, SW49 SW_Push, SW5 SW_Push, SW50 SW_Push, SW51 SW_Push, SW52 SW_Push, SW53 SW_Push, SW54 SW_Push, SW55 SW_Push, SW56 SW_Push, SW57 SW_Push, SW58 SW_Push, SW59 SW_Push, SW6 SW_Push, SW60 SW_Push, SW61 SW_Push, SW62 SW_Push, SW63 SW_Push, SW64 SW_Push, SW65 SW_Push, SW66 SW_Push, SW67 SW_Push, SW68 SW_Push, SW69 SW_Push, SW7 SW_Push, SW70 SW_Push, SW71 SW_Push, SW72 SW_Push, SW73 SW_Push, SW74 SW_Push, SW75 SW_Push, SW76 SW_Push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

Commit message: moved traces
Routing:
- net Net-(LED40-DOUT): track 0.00 -> 19.4 mm
- net Net-(LED39-DOUT): track 0.00 -> 17.9 mm
- net Net-(LED41-DOUT): track 0.00 -> 8.59 mm
Changed lines of the file:
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@@
+	)
+	(segment
+		(start 70.125 90.055)
+		(end 70.65 90.58)
+		(width 0.2)
+		(layer "B.Cu")
+		(net "Net-(LED39-DOUT)")
+	)
+	(segment
+		(start 71.57 93.57)
+		(end 82.42 93.57)
+		(width 0.2)
+		(layer "B.Cu")
+		(net "Net-(LED39-DOUT)")
+	)
+	(segment
+		(start 70.65 92.65)
+		(end 71.57 93.57)
+		(width 0.2)
+		(layer "B.Cu")
+		(net "Net-(LED39-DOUT)")
+	)
+	(segment
+		(start 82.42 93.57)
+		(end 83 92.99)
+		(width 0.2)
+		(layer "B.Cu")
+		(net "Net-(LED39-DOUT)")
+	)
+	(segment
+		(start 69.4 90.055)
+		(end 70.125 90.055)
+		(width 0.2)
+		(layer "B.Cu")
+		(net "Net-(LED39-DOUT)")
+	)
+	(segment
+		(start 70.65 90.58)
+		(end 70.65 92.65)
+		(width 0.2)
+		(layer "B.Cu")
+		(net "Net-(LED39-DOUT)")
+	)
+	(segment
+		(start 83 92.99)
+		(end 83 91.555)
+		(width 0.2)
+		(layer "B.Cu")
+		(net "Net-(LED39-DOUT)")
+	)
+	(segment
+		(start 90.04 93.5)
+		(end 90.7 94.16)
+		(width 0.2)
+		(layer "B.Cu")
+		(net "Net-(LED40-DOUT)")
+	)
+	(segment
+		(start 90.04 90.47)
+		(end 90.04 93.5)
+		(width 0.2)
+		(layer "B.Cu")
+		(net "Net-(LED40-DOUT)")
+	)
+	(segment
+		(start 90.7 94.16)
+		(end 101.62 94.16)
+		(width 0.2)
+		(layer "B.Cu")
+		(net "Net-(LED40-DOUT)")
+	)
+	(segment
+		(start 89.625 90.055)
+		(end 90.04 90.47)
+		(width 0.2)
+		(layer "B.Cu")
+		(net "Net-(LED40-DOUT)")
+	)
+	(segment
+		(start 88.45 90.055)
+		(end 89.625 90.055)
+		(width 0.2)
+		(layer "B.Cu")
+		(net "Net-(LED40-DOUT)")
+	)
+	(segment
+		(start 101.62 94.16)
+		(end 102.05 93.73)
+		(width 0.2)
+		(layer "B.Cu")
+		(net "Net-(LED40-DOUT)")
+	)
+	(segment
+		(start 102.05 91.555)
+		(end 102.05 93.73)
+		(width 0.2)
+		(layer "B.Cu")
+		(net "Net-(LED40-DOUT)")
+	)
+	(segment
+		(start 108.82 90.36)
+		(end 108.82 93.41)
+		(width 0.2)
+		(layer "B.Cu")
+		(net "Net-(LED41-DOUT)")
+	)
+	(segment
+		(start 112.69 93.81)
+		(end 112.73 93.77)
+		(width 0.2)
+		(layer "B.Cu")
+		(net "Net-(LED41-DOUT)")
+	)
+	(segment
+		(start 108.515 90.055)
+		(end 108.82 90.36)
+		(width 0.2)
+		(layer "B.Cu")
+		(net "Net-(LED41-DOUT)")
+	)
+	(segment
+		(start 107.5 90.055)
+		(end 108.515 90.055)
+		(width 0.2)
+		(layer "B.Cu")
+		(net "Net-(LED41-DOUT)")
+	)
+	(segment
+		(start 109.22 93.81)
+		(end 112.69 93.81)
+		(width 0.2)
+		(layer "B.Cu")
+		(net "Net-(LED41-DOUT)")
+	)
+	(segment
+		(start 108.82 93.41)
+		(end 109.22 93.81)
+		(width 0.2)
+		(layer "B.Cu")
+		(net "Net-(LED41-DOUT)")
 	)
 	(segment
