File: keeb.kicad_pcb (KiCad board)
At the start: 2 copper layers, 3.6 x 3.2 mm, 433 parts, among them SW1 SW_Push, SW10 SW_Push, SW100 SW_Push, SW101 SW_Push, SW102 SW_Push, SW103 SW_Push, SW104 SW_Push, SW105 SW_Push, SW11 SW_Push, SW12 SW_Push, SW13 SW_Push, SW14 SW_Push, SW15 SW_Push, SW16 SW_Push, SW17 SW_Push, SW18 SW_Push, SW19 SW_Push, SW2 SW_Push, SW20 SW_Push, SW21 SW_Push, SW22 SW_Push, SW23 SW_Push, SW24 SW_Push, SW25 SW_Push, SW26 SW_Push, SW27 SW_Push, SW28 SW_Push, SW29 SW_Push, SW3 SW_Push, SW30 SW_Push, SW31 SW_Push, SW32 SW_Push, SW33 SW_Push, SW34 SW_Push, SW35 SW_Push, SW36 SW_Push, SW37 SW_Push, SW38 SW_Push, SW39 SW_Push, SW4 SW_Push, SW40 SW_Push, SW41 SW_Push, SW42 SW_Push, SW43 SW_Push, SW44 SW_Push, SW45 SW_Push, SW46 SW_Push, SW47 SW_Push, SW48 SW_Push, SW49 SW_Push, SW5 SW_Push, SW50 SW_Push, SW51 SW_Push, SW52 SW_Push, SW53 SW_Push, SW54 SW_Push, SW55 SW_Push, SW56 SW_Push, SW57 SW_Push, SW58 SW_Push, SW59 SW_Push, SW6 SW_Push, SW60 SW_Push, SW61 SW_Push, SW62 SW_Push, SW63 SW_Push, SW64 SW_Push, SW65 SW_Push, SW66 SW_Push, SW67 SW_Push, SW68 SW_Push, SW69 SW_Push, SW7 SW_Push, SW70 SW_Push, SW71 SW_Push, SW72 SW_Push, SW73 SW_Push, SW74 SW_Push, SW75 SW_Push, SW76 SW_Push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

Commit message: did more work and journaling
Parts:
- moved U2 33.3 mm to (476.6, 143.1), turned to 180 degrees
Connections:
- A1 pad 11: /COL10 -> unconnected-(A1-GPIO8-Pad11)
- A1 pad 12: /COL11 -> unconnected-(A1-GPIO9-Pad12)
- A1 pad 14: /COL12 -> unconnected-(A1-GPIO10-Pad14)
- A1 pad 15: /COL13 -> unconnected-(A1-GPIO11-Pad15)
- A1 pad 16: /COL14 -> /ROTA
- A1 pad 17: /COL15 -> /ROTB
- A1 pad 19: /COL16 -> /ROTBU
- A1 pad 20: /COL17 -> /COL10
- A1 pad 21: /COL18 -> /COL9
- A1 pad 22: /COL19 -> /COL8
- A1 pad 24: /COL20 -> /COL7
- A1 pad 25: /ROTA -> /COL6
- A1 pad 26: /ROTB -> /COL5
- A1 pad 27: /ROTBU -> /COL4
- A1 pad 29: unconnected-(A1-GPIO22-Pad29) -> /COL3
- A1 pad 31: unconnected-(A1-GPIO26_ADC0-Pad31) -> /COL2
- A1 pad 32: unconnected-(A1-GPIO27_ADC1-Pad32) -> /COL1
- A1 pad 34: unconnected-(A1-GPIO28_ADC2-Pad34) -> /COL0
- U2 pad 1: /COL2 -> /COL18
- U2 pad 2: /COL3 -> /COL17
- U2 pad 27: /COL0 -> /COL20
- U2 pad 28: /COL1 -> /COL19
- U2 pad 3: /COL4 -> /COL16
- U2 pad 4: /COL5 -> /COL15
- U2 pad 5: /COL6 -> /COL14
- U2 pad 6: /COL7 -> /COL13
- U2 pad 7: /COL8 -> /COL12
- U2 pad 8: /COL9 -> /COL11
Routing:
- net /ROW1: track 0.00 -> 831.0 mm
- net /ROW2: track 0.00 -> 757.3 mm
- net /ROW4: track 0.00 -> 723.7 mm
- net /ROW3: track 0.00 -> 669.3 mm
- net /ROW5: track 0.00 -> 627.8 mm
- net /COL0: track 118.7 -> 679.9 mm
- net /COL1: track 139.1 -> 681.2 mm
- net /COL2: track 145.3 -> 657.2 mm
- net DIN: track 0.00 -> 510.8 mm
- net Net-(LED37-DOUT): track 0.00 -> 447.3 mm
- net /COL3: track 199.8 -> 630.5 mm
- net +5V: track 413.9 -> 0.00 mm, vias 4 -> 0
- net /COL8: track 128.2 -> 525.9 mm
- net Net-(LED16-DOUT): track 0.00 -> 387.9 mm
- net /COL10: track 137.6 -> 511.6 mm
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- added copper zone on B.Cu, net GND
