File: keeb.kicad_pcb (KiCad board)
At the start: 2 copper layers, 3.6 x 3.2 mm, 433 parts, among them SW1 SW_Push, SW10 SW_Push, SW100 SW_Push, SW101 SW_Push, SW102 SW_Push, SW103 SW_Push, SW104 SW_Push, SW105 SW_Push, SW11 SW_Push, SW12 SW_Push, SW13 SW_Push, SW14 SW_Push, SW15 SW_Push, SW16 SW_Push, SW17 SW_Push, SW18 SW_Push, SW19 SW_Push, SW2 SW_Push, SW20 SW_Push, SW21 SW_Push, SW22 SW_Push, SW23 SW_Push, SW24 SW_Push, SW25 SW_Push, SW26 SW_Push, SW27 SW_Push, SW28 SW_Push, SW29 SW_Push, SW3 SW_Push, SW30 SW_Push, SW31 SW_Push, SW32 SW_Push, SW33 SW_Push, SW34 SW_Push, SW35 SW_Push, SW36 SW_Push, SW37 SW_Push, SW38 SW_Push, SW39 SW_Push, SW4 SW_Push, SW40 SW_Push, SW41 SW_Push, SW42 SW_Push, SW43 SW_Push, SW44 SW_Push, SW45 SW_Push, SW46 SW_Push, SW47 SW_Push, SW48 SW_Push, SW49 SW_Push, SW5 SW_Push, SW50 SW_Push, SW51 SW_Push, SW52 SW_Push, SW53 SW_Push, SW54 SW_Push, SW55 SW_Push, SW56 SW_Push, SW57 SW_Push, SW58 SW_Push, SW59 SW_Push, SW6 SW_Push, SW60 SW_Push, SW61 SW_Push, SW62 SW_Push, SW63 SW_Push, SW64 SW_Push, SW65 SW_Push, SW66 SW_Push, SW67 SW_Push, SW68 SW_Push, SW69 SW_Push, SW7 SW_Push, SW70 SW_Push, SW71 SW_Push, SW72 SW_Push, SW73 SW_Push, SW74 SW_Push, SW75 SW_Push, SW76 SW_Push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

Commit message: did more routing
Connections:
- A1 pad 10: DIN -> unconnected-(A1-GPIO7-Pad10)
- A1 pad 15: unconnected-(A1-GPIO11-Pad15) -> /ROTA
- A1 pad 16: /ROTA -> /ROTB
- A1 pad 17: /ROTB -> /ROTBU
- A1 pad 19: /ROTBU -> DIN
- ROT_SW1 pad MP: unconnected-(ROT_SW1-PadMP) -> GND
Routing:
- net +5V: track 0.00 -> 1064.1 mm, vias 0 -> 1
- net Net-(LED58-DOUT): track 0.00 -> 461.2 mm
- net Net-(LED92-DOUT): track 0.00 -> 458.0 mm
- net Net-(LED74-DOUT): track 0.00 -> 434.2 mm
- net GND: track 0.00 -> 136.5 mm
- net Net-(LED71-DOUT): track 0.00 -> 109.0 mm
- net Net-(LED95-DOUT): track 0.00 -> 81.3 mm
- net Net-(LED96-DOUT): track 0.00 -> 76.1 mm
- net Net-(LED87-DOUT): track 0.00 -> 61.5 mm
- net Net-(LED88-DOUT): track 0.00 -> 42.9 mm
- net Net-(LED86-DOUT): track 0.00 -> 38.2 mm
- net Net-(LED103-DOUT): track 0.00 -> 32.6 mm
- net Net-(LED51-DOUT): track 0.00 -> 32.6 mm
- net Net-(LED50-DOUT): track 0.00 -> 32.6 mm
- net Net-(LED104-DOUT): track 0.00 -> 28.1 mm
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